File: RP2350b_40GPIO/KiCad/RP2350B_LevelShift.kicad_pcb (KiCad board)
At the start: 2 copper layers, 63.5 x 66.2 mm, 59 parts, among them J1 +5V, J10 SPI, J13 USB_B_Micro, J2 Right GPIO, J3 VGA, J4 Left GPIO, J7 SWD, J9 BOOT SEL, U1 LD1117S33TR_SOT223, U11 74CBTD3861, U12 74CBTD3861, U13 74CBTD3861, U14 74CBTD3861, U2 W25Q16JVSSIQ, U5 RP2350B-QFN80, U7 TLV74311PDBVR, Y1 12MHz

Commit message: - Added RP2350b_40GPIO Self Test Source Code.
Parts:
- C20, C21: value 8pf -> 10pf
- C22, C23, C24: footprint Capacitor_SMD:C_0805_2012Metric -> Capacitor_SMD:C_0603_1608Metric
- J13: footprint Dave Footprints:USB_Micro-B_Amphenol_10103594-0001LF_Horizontal -> _Custom:USB_Micro-B_Amphenol_10103594-0001LF_Horizontal
- J3: footprint SamacSys_Parts:117345301 -> _Custom:DSUB-15
- Power1: footprint SamacSys_Parts:LEDC2012X90N -> LED_SMD:LED_0805_2012Metric
- R20: value 1k -> 2k2
- U2: footprint Dave Footprints:SOIC-8_5.23x5.23mm_P1.27mm -> Package_SO:SOIC-8_5.3x5.3mm_P1.27mm
- U5: value RP2350B-QFN80 -> RP2354B-QFN80
Routing:
- net /2350_USB_D-: track 38.8 -> 38.2 mm
- net /2350_USB_D+: track 38.8 -> 38.3 mm
Other:
- board text added: "RP2354B Level Shifter 13/04/2025 Dave Gaunt."
- board text removed: "RP2350B Level Shifter 13/04/2025 Dave Gaunt."
